File: projeto1/projeto1.sch (KiCad schematic (older format))
At the start: 17 parts, among them J1 USB_B_Micro, J2 Conn_01x10, J3 Conn_01x10, J4 Conn_01x06, SW1 SW_Push, U1 ATmega32U4-AU, Y1 16MHz

Commit message: Processo de alocação dos componentes no PCB iniciado.
Connections:
- net Pino1: now reaches U1.1 (PE6)
- net Pino1: now also J2.10 (Pin_10); no longer J3.10 (Pin_10)
- net Pino10: now reaches U1.10 (PB2)
- net Pino10: now also J2.1 (Pin_1); no longer J2.3 (Pin_3)
- net Pino11: now reaches U1.11 (PB3)
- net Pino11: now also J4.1 (Pin_1); no longer J2.4 (Pin_4)
- net Pino12: now reaches U1.12 (PB7)
- net Pino12: now also J4.2 (Pin_2); no longer J2.8 (Pin_8)
- net Pino18: now reaches U1.18 (PD0)
- net Pino18: now also J4.3 (Pin_3); no longer J3.1 (Pin_1)
- net Pino19: now reaches U1.19 (PD1)
- net Pino19: now also J4.4 (Pin_4); no longer J3.2 (Pin_2)
- net Pino20: now reaches U1.20 (PD2)
- net Pino20: now also J4.5 (Pin_5); no longer J3.3 (Pin_3)
- net Pino21: now reaches U1.21 (PD3)
- net Pino21: now also J4.6 (Pin_6); no longer J3.4 (Pin_4)
- net Pino22: now reaches U1.22 (PD5)
- net Pino22: now also J3.1 (Pin_1); no longer J3.6 (Pin_6)
- net Pino25: now reaches U1.25 (PD4)
- net Pino25: now also J3.2 (Pin_2); no longer J3.5 (Pin_5)
- net Pino26: now reaches U1.26 (PD6)
- net Pino26: now also J3.3 (Pin_3); no longer J3.7 (Pin_7)
- net Pino27: now reaches U1.27 (PD7)
- net Pino27: now also J3.4 (Pin_4); no longer J3.8 (Pin_8)
- net Pino28: now reaches U1.28 (PB4)
- net Pino28: now also J3.5 (Pin_5); no longer J2.5 (Pin_5)
- net Pino29: now reaches U1.29 (PB5)
- net Pino29: now also J3.6 (Pin_6); no longer J2.6 (Pin_6)
- net Pino30: now reaches U1.30 (PB6)
- net Pino30: now also J3.7 (Pin_7); no longer J2.7 (Pin_7)
- net Pino31: now reaches U1.31 (PC6)
- net Pino31: now also J3.8 (Pin_8); no longer J2.9 (Pin_9)
- net Pino32: now reaches U1.32 (PC7)
- net Pino32: now also J3.9 (Pin_9); no longer J2.10 (Pin_10)
- net Pino33: now reaches U1.33 (~HWB~/PE2)
- net Pino33: now also J3.10 (Pin_10); no longer J3.9 (Pin_9)
- net Pino36: now reaches U1.36 (PF7)
- net Pino36: now also J2.9 (Pin_9); no longer J4.6 (Pin_6)
- net Pino37: now reaches U1.37 (PF6)
- net Pino37: now also J2.8 (Pin_8); no longer J4.5 (Pin_5)
- net Pino38: now reaches U1.38 (PF5)
- net Pino38: now also J2.7 (Pin_7); no longer J4.4 (Pin_4)
- net Pino39: now reaches U1.39 (PF4)
- net Pino39: now also J2.6 (Pin_6); no longer J4.3 (Pin_3)
- net Pino40: now reaches U1.40 (PF1)
- net Pino40: now also J2.5 (Pin_5); no longer J4.2 (Pin_2)
- net Pino41: now reaches U1.41 (PF0)
- net Pino41: now also J2.4 (Pin_4); no longer J4.1 (Pin_1)
- net Pino8: now reaches U1.8 (PB0)
- net Pino8: now also J2.3 (Pin_3); no longer J2.1 (Pin_1)
- net Pino9: now reaches J2.2 (Pin_2), U1.9 (PB1)
Other:
- moved on the sheet: J2, J3, J4
